File: froggy.sch (KiCad schematic (older format))
At the start: 14 parts, among them J1 USB_C_Receptacle_USB2.0, J2 Micro_SD_Card, U1 FT232RL, U2 LEAPSTER-CART

Commit message: [upload] beautification
Parts:
- C1, C2, C3, C4: footprint (none) -> Capacitor_SMD:C_0603_1608Metric
- D1, D2: footprint (none) -> Diode_SMD:D_0603_1608Metric
- J1: footprint (none) -> Connector_USB:USB_C_Receptacle_GCT_USB4085
- J2: footprint (none) -> SamacSys_Parts:5040771891
- R1, R2, R3, R4: footprint (none) -> Resistor_SMD:R_0603_1608Metric
- U2: footprint (none) -> Leapster:LEAPSTER_CART
Connections:
- net D0 is gone; now on net +3V3: U2.25 (3V3)
- net D1 is gone; now on net CLK: U2.24 (SD_CLK)
- net L_RXD is gone; now on net L_RX: R3.1
- net L_TXD is gone; now on net L_TX: R4.2
- net +3V3: now also U2.8 (3V3); no longer U2.18 (GND), U2.28 (SD_D3)
- net CLK: no longer U2.27 (SD_CMD)
- net CMD: now also U2.27 (SD_CMD)
- net DAT0: now also U2.22 (SD_D0)
- net DAT1: now also U2.21 (SD_D1)
- net DAT2: now also U2.29 (SD_D2)
- net DAT3: now also U2.28 (SD_D3)
- net GND: now also U2.18 (GND), U2.23 (GND), U2.9 (GND); no longer U2.19 (TX), U2.29 (SD_D2)
- net L_RX: now also U2.20 (RX)
- net L_TX: now also U2.19 (TX)
- no-connect marks 4 -> 16
Other:
- moved on the sheet: C1, C2, C3, C4, D1, D2, J1, J2, R1, R2, R3, R4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

Commit message: [tweak] uploading the working tested version
Parts:
- added R5: 1K, Resistor_SMD:R_0603_1608Metric, symbol Device:R
- added R6: 2K, Resistor_SMD:R_0603_1608Metric, symbol Device:R
Connections:
- net +5V: now also R5.1; no longer D2.2 (A)
- net GND: now also U2.30 (A18), R6.2
- new net: D2.2 (A), R5.2, R6.1
- no-connect marks 16 -> 32
Other:
- moved on the sheet: D2
Changed lines of the file:
@@
 L power:GND #PWR0101
 U 1 1 5FE10448
-P 3950 4750
-F 0 "#PWR0101" H 3950 4500 50  0001 C CNN
-F 1 "GND" V 3955 4622 50  0000 R CNN
-F 2 "" H 3950 4750 50  0001 C CNN
-F 3 "" H 3950 4750 50  0001 C CNN
-	1    3950 4750
-	0    1    1    0
+P 4100 5250
+F 0 "#PWR0101" H 4100 5000 50  0001 C CNN
+F 1 "GND" V 4105 5122 50  0000 R CNN
+F 2 "" H 4100 5250 50  0001 C CNN
+F 3 "" H 4100 5250 50  0001 C CNN
+	1    4100 5250
+	1    0    0    -1
 $EndComp
 $Comp
 L power:+5V #PWR0102
 U 1 1 5FE0FB3B
-P 4250 4750
-F 0 "#PWR0102" H 4250 4600 50  0001 C CNN
-F 1 "+5V" V 4265 4878 50  0000 L CNN
-F 2 "" H 4250 4750 50  0001 C CNN
-F 3 "" H 4250 4750 50  0001 C CNN
-	1    4250 4750
+P 4550 4950
+F 0 "#PWR0102" H 4550 4800 50  0001 C CNN
+F 1 "+5V" V 4565 5078 50  0000 L CNN
+F 2 "" H 4550 4950 50  0001 C CNN
+F 3 "" H 4550 4950 50  0001 C CNN
+	1    4550 4950
 	0    1    1    0
 $EndComp
@@
 L Device:LED D2
 U 1 1 5FE0E815
-P 4100 4750
-F 0 "D2" H 4093 4967 50  0000 C CNN
-F 1 "USB_INSERTED_LED" H 4093 4876 50  0000 C CNN
-F 2 "Diode_SMD:D_0603_1608Metric" H 4100 4750 50  0001 C CNN
-F 3 "~" H 4100 4750 50  0001 C CNN
-	1    4100 4750
-	1    0    0    -1
+P 4100 5100
+F 0 "D2" H 4093 5317 50  0000 C CNN
+F 1 "USB_INSERTED_LED" H 4093 5226 50  0000 C CNN
+F 2 "Diode_SMD:D_0603_1608Metric" H 4100 5100 50  0001 C CNN
+F 3 "~" H 4100 5100 50  0001 C CNN
+	1    4100 5100
+	0    -1   -1   0
 $EndComp
 $Comp
 L power:GND #PWR0103
 U 1 1 5FE0CF14
-P 3950 4400
-F 0 "#PWR0103" H 3950 4150 50  0001 C CNN
-F 1 "GND" V 3955 4272 50  0000 R CNN
-F 2 "" H 3950 4400 50  0001 C CNN
-F 3 "" H 3950 4400 50  0001 C CNN
-	1    3950 4400
-	0    1    1    0
+P 3650 4400
+F 0 "#PWR0103" H 3650 4150 50  0001 C CNN
+F 1 "GND" V 3655 4272 50  0000 R CNN
+F 2 "" H 3650 4400 50  0001 C CNN
+F 3 "" H 3650 4400 50  0001 C CNN
+	1    3650 4400
+	1    0    0    -1
 $EndComp
 $Comp
@@
 P 3650 3800
 F 0 "#PWR0114" H 3650 3550 50  0001 C CNN
-F 1 "GND" V 3655 3672 50  0000 R CNN
+F 1 "GND" V 3650 3650 50  0000 R CNN
 F 2 "" H 3650 3800 50  0001 C CNN
 F 3 "" H 3650 3800 50  0001 C CNN
 	1    3650 3800
-	0    -1   -1   0
+	1    0    0    -1
 $EndComp
 Connection ~ 3350 3800
@@
 	1    0    0    -1
 $EndComp
-Connection ~ 4650 2500
 Wire Wire Line
 	4650 2600 4650 2500
@@
 L power:GND #PWR0116
 U 1 1 5FDC46FF
-P 4650 2500
-F 0 "#PWR0116" H 4650 2250 50  0001 C CNN
-F 1 "GND" V 4655 2372 50  0000 R CNN
-F 2 "" H 4650 2500 50  0001 C CNN
-F 3 "" H 4650 2500 50  0001 C CNN
-	1    4650 2500
-	0    -1   -1   0
+P 4650 2600
+F 0 "#PWR0116" H 4650 2350 50  0001 C CNN
+F 1 "GND" V 4655 2472 50  0000 R CNN
+F 2 "" H 4650 2600 50  0001 C CNN
+F 3 "" H 4650 2600 50  0001 C CNN
+	1    4650 2600
+	1    0    0    -1
 $EndComp
 $Comp
@@
 F 3 "" H 4250 2050 50  0001 C CNN
 	1    4250 2050
-	0    -1   -1   0
+	1    0    0    -1
 $EndComp
 $Comp
@@
 F 3 "" H 5100 1750 50  0001 C CNN
 	1    5100 1750
-	0    1    1    0
+	1    0    0    -1
 $EndComp
 Wire Wire Line
@@
 	0    -1   -1   0
 $EndComp
+$Comp
+L power:GND #PWR0124
+U 1 1 5FEC0C19
+P 8650 5100
+F 0 "#PWR0124" H 8650 4850 50  0001 C CNN
+F 1 "GND" V 8655 4972 50  0000 R CNN
+F 2 "" H 8650 5100 50  0001 C CNN
+F 3 "" H 8650 5100 50  0001 C CNN
+	1    8650 5100
+	0    -1   -1   0
+$EndComp
+Connection ~ 4650 2600
+Wire Wire Line
+	3650 4400 3950 4400
+NoConn ~ 8650 3300
+NoConn ~ 8650 3400
+NoConn ~ 8650 3500
+NoConn ~ 8650 3600
+NoConn ~ 8650 3700
+NoConn ~ 8650 3800
+NoConn ~ 8650 3900
+NoConn ~ 8650 4200
+NoConn ~ 8650 4300
+NoConn ~ 8650 4400
+NoConn ~ 8650 4500
+NoConn ~ 8650 4600
+NoConn ~ 8650 4700
+NoConn ~ 8650 4800
+NoConn ~ 8650 4900
+NoConn ~ 5400 2450
+$Comp
+L Device:R R5
+U 1 1 5FF28926
+P 4400 4950
+F 0 "R5" V 4193 4950 50  0000 C CNN
+F 1 "1K" V 4284 4950 50  0000 C CNN
+F 2 "Resistor_SMD:R_0603_1608Metric" V 4330 4950 50  0001 C CNN
+F 3 "~" H 4400 4950 50  0001 C CNN
+	1    4400 4950
+	0    1    1    0
+$EndComp
+Wire Wire Line
+	4250 4950 4100 4950
+$Comp
+L Device:R R6
+U 1 1 5FF2F190
+P 3750 4950
+F 0 "R6" V 3543 4950 50  0000 C CNN
+F 1 "2K" V 3634 4950 50  0000 C CNN
+F 2 "Resistor_SMD:R_0603_1608Metric" V 3680 4950 50  0001 C CNN
+F 3 "~" H 3750 4950 50  0001 C CNN
+	1    3750 4950
+	0    1    1    0
+$EndComp
+Wire Wire Line
+	3900 4950 4100 4950
+Connection ~ 4100 4950
+$Comp
+L power:GND #PWR0125
+U 1 1 5FF32F3E
+P 3600 4950
+F 0 "#PWR0125" H 3600 4700 50  0001 C CNN
+F 1 "GND" H 3605 4777 50  0000 C CNN
+F 2 "" H 3600 4950 50  0001 C CNN
+F 3 "" H 3600 4950 50  0001 C CNN
+	1    3600 4950
+	1    0    0    -1
+$EndComp
 $EndSCHEMATC
